Commit message: gripper urdf configs for holder vs gripper

File: robotiq_description/urdf/robotiq_hand_e_macro.urdf.xacro (robot description, xacro)
@@ -16,4 +16,6 @@
                  right_finger_scale:=default right_finger_collision_scale:=default
                  tcp_z_offset:=0.1325
+                 enable_collisions:=true
+                 joint_type:=prismatic
                  ">
       <xacro:property name="file_path" value="file://$(find robotiq_description)" />
@@ -50,18 +52,20 @@
             <inertia ixx="1017560E-9" ixy="0" ixz="2235E-9" iyy="1028041E-9" iyz="0" izz="489810E-9"/>
           </inertial>
-          <visual>
-              <origin rpy="0 0 0" xyz="0 0 0"/>
-              <geometry>
-                  <mesh filename="${file_path}/meshes/visual/hande/hand-e.dae" scale="1.0 1.0 1.0"/>
-              </geometry>
-              <material name="dark" />
-          </visual>
-          <collision>
-              <origin rpy="0 0 0" xyz="0 0 0"/>
-              <geometry>
-                  <mesh filename="${file_path}/meshes/collision/hande/hand-e.stl" scale="1.0 1.0 1.0"/>
-                  <!--<mesh filename="${file_path}/meshes/collision/hande/hand-e_convex_hull.stl" scale="1.0 1.0 1.0"/>-->
-              </geometry>
-          </collision>
+          <xacro:if value="${enable_collisions}">
+            <visual>
+                <origin rpy="0 0 0" xyz="0 0 0"/>
+                <geometry>
+                    <mesh filename="${file_path}/meshes/visual/hande/hand-e.dae" scale="1.0 1.0 1.0"/>
+                </geometry>
+                <material name="dark" />
+            </visual>
+            <collision>
+                <origin rpy="0 0 0" xyz="0 0 0"/>
+                <geometry>
+                    <mesh filename="${file_path}/meshes/collision/hande/hand-e.stl" scale="1.0 1.0 1.0"/>
+                    <!--<mesh filename="${file_path}/meshes/collision/hande/hand-e_convex_hull.stl" scale="1.0 1.0 1.0"/>-->
+                </geometry>
+            </collision>
+          </xacro:if>
       </link>
       <joint name="${prefix}robotiq_hande_base_joint" type="fixed">
@@ -72,38 +76,42 @@
       <!-- Fingers -->
       <link name="${prefix}hande_left_finger">
-          <visual>
-            <origin rpy="0 0 0" xyz="0 0 0"/>
-            <geometry>
-              <mesh filename="${left_finger_visual}" scale="${left_finger_scale}" />
-            </geometry>
-            <material name="gray">
-              <color rgba="0.7 0.7 0.7 1.0"/>
-            </material>
-          </visual>
-          <collision>
-            <origin rpy="0 0 0" xyz="${-0.010} ${-0.075/2} ${0.028/2}"/>
-            <geometry>
-<!--               <mesh filename="${left_finger_collision}" scale="1.0 1.0 1.0" /> -->
-              <box size="${left_finger_collision_scale}" />
-            </geometry>
-          </collision>
+          <xacro:if value="${enable_collisions}">
+            <visual>
+              <origin rpy="0 0 0" xyz="0 0 0"/>
+              <geometry>
+                <mesh filename="${left_finger_visual}" scale="${left_finger_scale}" />
+              </geometry>
+              <material name="gray">
+                <color rgba="0.7 0.7 0.7 1.0"/>
+              </material>
+            </visual>
+            <collision>
+              <origin rpy="0 0 0" xyz="${-0.010} ${-0.075/2} ${0.028/2}"/>
+              <geometry>
+  <!--               <mesh filename="${left_finger_collision}" scale="1.0 1.0 1.0" /> -->
+                <box size="${left_finger_collision_scale}" />
+              </geometry>
+            </collision>
+          </xacro:if>
         </link>
         <link name="${prefix}hande_right_finger">
-          <visual>
-            <origin rpy="0 0 0" xyz="0 0 0"/>
-            <geometry>
-              <mesh filename="${right_finger_visual}" scale="${right_finger_scale}" />
-            </geometry>
-            <material name="gray">
-              <color rgba="0.7 0.7 0.7 1.0"/>
-            </material>
-          </visual>
-          <collision>
-            <origin rpy="0 0 0" xyz="${0.010} ${-0.075/2} ${0.028/2}"/>
-            <geometry>
-              <box size="${right_finger_collision_scale}" />
-<!--               <mesh filename="${right_finger_collision}" scale="1.0 1.0 1.0" /> -->
-            </geometry>
-          </collision>
+          <xacro:if value="${enable_collisions}">
+            <visual>
+              <origin rpy="0 0 0" xyz="0 0 0"/>
+              <geometry>
+                <mesh filename="${right_finger_visual}" scale="${right_finger_scale}" />
+              </geometry>
+              <material name="gray">
+                <color rgba="0.7 0.7 0.7 1.0"/>
+              </material>
+            </visual>
+            <collision>
+              <origin rpy="0 0 0" xyz="${0.010} ${-0.075/2} ${0.028/2}"/>
+              <geometry>
+                <box size="${right_finger_collision_scale}" />
+  <!--               <mesh filename="${right_finger_collision}" scale="1.0 1.0 1.0" /> -->
+              </geometry>
+            </collision>
+          </xacro:if>
       </link>
       <!-- virtual joint to model values coming from the gripper to the geometry - gripper uses
@@ -118,5 +126,5 @@
         <limit effort="180" lower="0.0" upper="${gripper_maximal_stroke}" velocity="0.15"/>
       </joint>
-      <joint name="${prefix}hande_left_finger_joint" type="prismatic">
+      <joint name="${prefix}hande_left_finger_joint" type="${joint_type}">
         <origin rpy="0 0 0" xyz="0 0 0.099"/>
         <parent link="${prefix}hand_e_base_link"/>
@@ -126,5 +134,5 @@
         <mimic joint="${prefix}hande_finger_distance" multiplier="-0.5" offset="${gripper_maximal_stroke/2}"/>
       </joint>
-      <joint name="${prefix}hande_right_finger_joint" type="prismatic">
+      <joint name="${prefix}hande_right_finger_joint" type="${joint_type}">
         <origin rpy="0 0 0" xyz="0 0 0.099"/>
         <parent link="${prefix}hand_e_base_link"/>
@@ -134,9 +142,9 @@
         <mimic joint="${prefix}hande_finger_distance" multiplier="-0.5" offset="${gripper_maximal_stroke/2}"/>
       </joint>
-      <link name="$(arg prefix)tcp_link"/>
-      <joint name="$(arg prefix)tcp_link_joint" type="fixed">
+      <link name="${prefix}tcp_link"/>
+      <joint name="${prefix}tcp_link_joint" type="fixed">
         <origin xyz="0 0 ${tcp_z_offset}" rpy="0 0 ${-pi/2}"/>
-        <parent link="$(arg prefix)hand_e_base_link"/>
-        <child link="$(arg prefix)tcp_link"/>
+        <parent link="${prefix}hand_e_base_link"/>
+        <child link="${prefix}tcp_link"/>
       </joint>
     </xacro:macro>
